Commit message: 模拟预览

File: install/dh_gripper_description/share/dh_gripper_description/urdf/ag95_macro.xacro (robot description, xacro)
@@ -1,5 +1,4 @@
 <?xml version="1.0"?>
 <robot xmlns:xacro="http://www.ros.org/wiki/xacro">
-  <xacro:property name="pi" value="3.14159265" />
   <xacro:macro name="dh_ag95_gripper" params="prefix parent">
     <joint name="${prefix}gripper_base_joint" type="fixed">
